Commit message: walk

File: qwe.SLDASM/urdf/qwe.SLDASM.urdf (robot description, URDF)
Before this commit: robot qwe_dog, 13 links, 12 joints
Joints:
- joint shank_front_left_joint: limit lower=-1.396 upper=1.396 effort=1.27 velocity=6.3 -> lower=-1.57 upper=1.57 effort=1.27 velocity=6.3
- joint shank_front_right_joint: limit lower=-1.396 upper=1.396 effort=1.27 velocity=6.3 -> lower=-1.57 upper=1.57 effort=1.27 velocity=6.3
- joint shank_rear_left_joint: limit lower=-1.396 upper=1.396 effort=1.27 velocity=6.3 -> lower=-1.57 upper=1.57 effort=1.27 velocity=6.3
- joint shank_rear_right_joint: limit lower=-1.396 upper=1.396 effort=1.27 velocity=6.3 -> lower=-1.57 upper=1.57 effort=1.27 velocity=6.3
- joint thigh_front_left_joint: limit lower=-0.6 upper=0.6 effort=1.27 velocity=6.3 -> lower=-1.4 upper=1.4 effort=1.27 velocity=6.3
- joint thigh_front_right_joint: limit lower=-0.6 upper=0.6 effort=1.27 velocity=6.3 -> lower=-1.4 upper=1.4 effort=1.27 velocity=6.3
- joint thigh_rear_left_joint: limit lower=-0.6 upper=0.6 effort=1.27 velocity=6.3 -> lower=-1.4 upper=1.4 effort=1.27 velocity=6.3
- joint thigh_rear_right_joint: limit lower=-0.6 upper=0.6 effort=1.27 velocity=6.3 -> lower=-1.4 upper=1.4 effort=1.27 velocity=6.3
